File: Swadge-HW/Swadge-HW.kicad_pcb (KiCad board)
At the start: 2 copper layers, 304.8 x 149.9 mm, 99 parts, among them J1 SAO, J2 PJ-307C, J3 PGM, P1 USB_C_Plug_USB2.0, Q1 Q_PMOS_GSD, SW1 YTS-D003-1A, SW2 YTS-D003-1A, SW3 YTS-D003-1A, SW4 YTS-D003-1A, SW5 YTS-D003-1A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

Commit message: longdog
longdog layout
Parts:
- removed the REF** at (87.3, 124.5)
- removed the REF** at (227.3, 124.5)
- moved R17 149.5 mm to (341.5, 143.9)
- moved D9 148.6 mm to (351.4, 191.7), turned to 133 degrees
- moved SW8 148.1 mm to (338.6, 122.7)
- moved SW7 148.1 mm to (327.0, 128.2)
- moved R15 147.5 mm to (345.7, 153.5)
- moved D11 145.7 mm to (311.9, 195.9)
- moved P1 145.7 mm to (316.0, 204.4)
- moved R27 145.7 mm to (315.5, 196.0)
- moved D12 145.7 mm to (308.3, 199.2)
- moved R13 145.7 mm to (317.4, 196.5)
- moved R14 145.7 mm to (319.3, 197.0)
- moved R28 145.7 mm to (321.3, 197.6)
- moved R11 141.2 mm to (336.0, 133.4)
- moved U4 140.9 mm to (346.3, 164.1)
- moved R10 139.4 mm to (352.5, 133.6)
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
Commit message: art adjustment
Parts:
- moved C3 115.2 mm to (291.8, 80.7)
- moved C2 115.2 mm to (292.0, 79.2)
- moved R19 58.6 mm to (182.6, 79.7)
- moved BT2 0.69 mm to (234.0, 124.2)
Routing:
- net USB_D-: track 0.00 -> 117.4 mm
- net USB_D+: track 0.00 -> 116.7 mm
- net SPK_SHDN: track 0.00 -> 110.1 mm, vias 0 -> 2
- net SPK: track 0.00 -> 103.7 mm, vias 0 -> 2
- net Net-(U9-+): track 0.00 -> 41.0 mm, vias 0 -> 1
- net LCD28: track 0.00 -> 38.0 mm, vias 0 -> 1
- net TFTATP: track 0.00 -> 36.4 mm
- net EN: track 0.00 -> 34.4 mm
- net TFT_RS: track 0.00 -> 19.5 mm, vias 0 -> 1
- net Net-(U8-IN-): track 0.00 -> 16.5 mm, vias 0 -> 2
- net 5VIN: track 0.00 -> 15.4 mm, vias 0 -> 2
- net Net-(U8-VO2): track 0.00 -> 13.7 mm
- net Net-(U8-VO1): track 0.00 -> 12.8 mm, vias 0 -> 2
- net Net-(J2-Pad1): track 0.00 -> 12.3 mm, vias 0 -> 1
- net Net-(P1-DN1): track 0.00 -> 12.0 mm, vias 0 -> 2
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
Commit message: shape and routing
Parts:
- moved REF** 102.5 mm to (279.3, 139.5)
- moved R27 45.4 mm to (284.5, 162.8)
- moved D11 45.4 mm to (280.9, 162.7)
- moved D12 45.4 mm to (277.3, 166.0)
- moved R13 45.4 mm to (286.4, 163.3)
- moved R14 45.4 mm to (288.4, 163.8)
- moved R28 45.4 mm to (290.3, 164.3)
- moved SW7 44.4 mm to (335.1, 171.8)
- moved SW8 44.4 mm to (346.7, 166.3)
- moved P1 43.6 mm to (286.8, 172.1), turned to 172 degrees
- moved R10 42.5 mm to (379.0, 166.9)
- moved R15 42.5 mm to (372.2, 186.8)
- moved R16 42.5 mm to (381.2, 180.1)
- moved R12 42.5 mm to (357.1, 181.4)
- moved R17 42.5 mm to (368.0, 177.2)
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Routing:
- net +5V: track 0.00 -> 145.6 mm
- net SPK_SHDN: track 110.1 -> 1.64 mm, vias 2 -> 0
- net +3V3: track 11.5 -> 94.6 mm, vias 0 -> 8
- net USB_D-: track 117.4 -> 47.3 mm, vias 0 -> 2
- net USB_D+: track 116.7 -> 47.1 mm, vias 0 -> 2
- net TFT_FMARK: track 0.00 -> 69.0 mm, vias 0 -> 1
- net TFT_SCL: track 0.00 -> 68.8 mm, vias 0 -> 3
- net TFT_CS: track 0.00 -> 65.0 mm, vias 0 -> 1
- net 5VIN: track 15.4 -> 78.0 mm
- net TFT_SDA: track 0.00 -> 60.5 mm, vias 0 -> 1
- net TFT_RESET: track 0.00 -> 57.5 mm, vias 0 -> 1
- net LED: track 0.00 -> 49.4 mm, vias 0 -> 2
- net Net-(U8-VO1): track 12.8 -> 43.1 mm
- net Net-(U8-VO2): track 13.7 -> 38.9 mm
- net Net-(U8-IN-): track 16.5 -> 37.4 mm
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Other:
- board size 304.8 x 149.9 mm -> 305 x 100.2 mm
- board text added: "A"
- board text added: "B"

Commit message: Update Swadge-HW.kicad_pcb
Parts:
- moved R16 0.86 mm to (380.3, 180.0)
Routing:
- net +3V3: track 94.6 -> 614.6 mm, vias 8 -> 27
- net BTN_1: track 0.00 -> 243.9 mm, vias 0 -> 8
- net BTN_3: track 0.00 -> 226.9 mm, vias 0 -> 7
- net BTN_4: track 0.00 -> 225.9 mm, vias 0 -> 9
- net BTN_2: track 0.00 -> 220.9 mm, vias 0 -> 7
- net VMON: track 0.00 -> 180.0 mm, vias 0 -> 4
- net SDA: track 13.1 -> 176.6 mm, vias 0 -> 3
- net SCL: track 13.0 -> 172.9 mm, vias 2 -> 4
- net BTN_5: track 0.00 -> 148.5 mm, vias 0 -> 5
- net BTN_6: track 0.00 -> 122.9 mm, vias 0 -> 5
- net TOUCH_6: track 0.00 -> 118.9 mm, vias 0 -> 2
- net TOUCH_4: track 0.00 -> 114.7 mm, vias 0 -> 2
- net TOUCH_3: track 0.00 -> 104.6 mm, vias 0 -> 4
- net TOUCH_1: track 0.00 -> 103.9 mm, vias 0 -> 2
- net TOUCH_5: track 0.00 -> 101.6 mm, vias 0 -> 2
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- added copper zone on B.Cu, net GND
- added copper zone on F.Cu, net GND
