File: Swadge-HW/Swadge-HW.kicad_pcb (KiCad board)
At the start: 2 copper layers, 305 x 100.2 mm, 97 parts, among them J1 SAO, J2 PJ-307C, J3 PGM, P1 USB_C_Plug_USB2.0, Q1 Q_PMOS_GSD, SW1 YTS-D003-1A, SW2 YTS-D003-1A, SW3 YTS-D003-1A, SW4 YTS-D003-1A, SW5 YTS-D003-1A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

Commit message: Update Swadge-HW.kicad_pcb
Routing:
- net +3V3: track 614.6 -> 614.5 mm, vias 27 -> 25

Commit message: generated mfg files for quoting
Routing:
- net BTN_8: track 93.9 -> 111.0 mm
- net BTN_7: track 88.1 -> 103.0 mm, vias 3 -> 1
- net GND: track 36.7 -> 43.7 mm, vias 9 -> 139
- net Net-(D4-OUT): track 57.5 -> 64.0 mm
- net LED: track 49.2 -> 53.7 mm
- net TOUCH_4: track 114.7 -> 118.9 mm
- net +3V3: track 614.5 -> 618.0 mm, vias 25 -> 22
- net SPK: track 83.6 -> 86.2 mm, vias 4 -> 2
- net SCL: track 172.9 -> 170.6 mm
- net MIC: track 39.3 -> 36.9 mm, vias 5 -> 4
- net BTN_1: track 243.9 -> 245.8 mm, vias 8 -> 6
- net VMON: track 180.0 -> 181.9 mm, vias 4 -> 2
- net BTN_6: track 122.9 -> 121.1 mm
- net BTN_4: track 225.9 -> 224.3 mm, vias 9 -> 7
- net BTN_2: track 220.9 -> 219.5 mm, vias 7 -> 5
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